Commit message: new urdf

File: src/p3dx_description/urdf/pioneer3dx.xacro (robot description, xacro)
@@ -203,5 +203,5 @@
    <joint name="chassis_to_rplidar" type="fixed">
      <axis xyz="0 0 0" />
-     <origin rpy="0 0 -1.57" xyz="0.06 0.0 0.33" />
+     <origin rpy="0 0 -1.57" xyz="0.065 0.0 0.339" />
      <parent link="chassis" />
      <child link="rplidar" />
@@ -223,5 +223,5 @@
 			parent="chassis" child="rplidar" /> -->
 	<xacro:sensor_d435 parent="chassis">
-		<origin xyz="0.1 0 0.860" rpy="0 0 0"/>
+		<origin xyz="0.16 0 0.670" rpy="0 0 0"/>
     </xacro:sensor_d435>
 	<!-- <xacro:sensor_d455 parent="chassis" use_nominal_extrinsics="$(arg use_nominal_extrinsics)">

Commit message: Stable

File: src/p3dx_description/urdf/pioneer3dx.xacro (robot description, xacro)
@@ -16,21 +16,12 @@
 work original in ucs-ros-pkg.
  -->
-<robot name="pioneer3dx" xmlns:xacro="http://ros.org/wiki/xacro">
-  <!-- import all gazebo-customization elements, including gazebo colors -->
-  	<xacro:include filename="$(find p3dx_description)/urdf/pioneer3dx.gazebo" />
-  <!-- import the pioneer 3dx's wheels -->
-  	<xacro:include filename="$(find p3dx_description)/urdf/pioneer3dx_wheel.xacro" />
-  	<xacro:include filename="$(find p3dx_description)/urdf/_d435.xacro" />
-  	<!-- <xacro:include filename="$(find realsense2_description)/urdf/_d455.urdf.xacro" /> -->
-  <!-- <xacro:include filename="$(find p3dx_description)/urdf/_d435.gazebo.xacro" /> -->
-	<xacro:arg name="use_nominal_extrinsics" default="false"/>
-  	<link name="base_link"/>
-    <joint name="dummy_joint" type="fixed">
-      <parent link="base_link"/>
-      <child link="chassis" />
-      <origin xyz="0 0 0.0" rpy="0 0 0"/>
-    </joint>
-  <!-- chassis -->
-	<link name="chassis">
+<robot name="pioneer3dx"
+	xmlns:xacro="http://ros.org/wiki/xacro">
+	<!-- import all gazebo-customization elements, including gazebo colors -->
+	<xacro:include filename="$(find p3dx_description)/urdf/pioneer3dx.gazebo" />
+	<!-- import the pioneer 3dx's wheels -->
+	<xacro:include filename="$(find p3dx_description)/urdf/pioneer3dx_wheel.xacro" />
+	<!-- chassis -->
+	<link name="base_link">
 		<inertial>
 			<mass value="3.5" />
@@ -39,12 +30,10 @@
 			<inertia ixx="1" ixy="0" ixz="0" iyy="1" iyz="0" izz="1" />
 		</inertial>
-		<visual name="base_visual">
+		<visual>
 			<origin xyz="-0.045 0 0.148" rpy="0 0 0" />
 			<geometry name="pioneer_geom">
 				<mesh filename="package://p3dx_description/meshes/chassis.stl" />
 			</geometry>
-			<material name="ChassisRed">
-				<color rgba="0.851 0.0 0.0 1.0" />
-			</material>
+			<material name="ChassisRed"></material>
 		</visual>
 		<collision>
@@ -55,5 +44,5 @@
 		</collision>
 	</link>
-  <!-- top_plate -->
+	<!-- top_plate -->
 	<link name="top_plate">
 		<inertial>
@@ -62,12 +51,10 @@
 			<inertia ixx="1" ixy="0" ixz="0" iyy="1" iyz="0" izz="1" />
 		</inertial>
-		<visual name="base_visual">
+		<visual>
 			<origin xyz="0 0 0" rpy="0 0 0" />
 			<geometry name="top_geom">
 				<mesh filename="package://p3dx_description/meshes/top.stl" />
 			</geometry>
-			<material name="TopBlack">
-				<color rgba="0.038 0.038 0.038 1.0" />
-			</material>
+			<material name="TopBlack"></material>
 		</visual>
 		<collision>
@@ -80,8 +67,8 @@
 	<joint name="base_top_joint" type="fixed">
 		<origin xyz="-0.045 0 0.234" rpy="0 0 0" />
-		<parent link="chassis" />
+		<parent link="base_link" />
 		<child link="top_plate" />
 	</joint>
-  <!-- swivel -->
+	<!-- swivel -->
 	<link name="swivel">
 		<inertial>
@@ -90,21 +77,19 @@
 			<inertia ixx="0.01" ixy="0" ixz="0" iyy="0.01" iyz="0" izz="0.01" />
 		</inertial>
-		<visual name="base_visual">
+		<visual>
 			<origin xyz="0 0 0" rpy="0 0 0" />
 			<geometry name="pioneer_geom">
 				<mesh filename="package://p3dx_description/meshes/swivel.stl" />
 			</geometry>
-			<material name="swivel">
-				<color rgba="0.5 0.5 0.5 1" />
-			</material>
-		</visual>
-		<collision>
-			<origin xyz="0 0 0" rpy="0 0 0" />
-			<geometry>
-				<box size="0 0 0" />
-			</geometry>
-		</collision>
-	</link>
-	<joint name="base_swivel_joint" type="continuous">
+			<material name="swivel"></material>
+		</visual>
+		<collision>
+			<origin xyz="0 0 0" rpy="0 0 0" />
+			<geometry>
+				<box size="0.00001 0.00001 0.00001" />
+			</geometry>
+		</collision>
+	</link>
+	<joint name="base_swivel_joint" type="fixed">
 		<origin xyz="-0.185 0 0.055" rpy="0 0 0" />
 		<axis xyz="0 0 1" />
@@ -112,32 +97,29 @@
 		<limit effort="100" velocity="100" k_velocity="0" />
 		<joint_properties damping="0.0" friction="0.0" />
-		<parent link="chassis" />
+		<parent link="base_link" />
 		<child link="swivel" />
 	</joint>
-  <!-- center_hubcap -->
+	<!-- center_hubcap -->
 	<link name="center_hubcap">
 		<inertial>
 			<mass value="0.01" />
 			<origin xyz="0 0 0" />
-			<inertia ixx="0.012411765597" ixy="-0.000711733678" ixz="0.00050272983"
-				iyy="0.015218160428" iyz="-0.000004273467" izz="0.011763977943" />
-		</inertial>
-		<visual name="base_visual">
+			<inertia ixx="0.012411765597" ixy="-0.000711733678" ixz="0.00050272983" iyy="0.015218160428" iyz="-0.000004273467" izz="0.011763977943" />
+		</inertial>
+		<visual>
 			<origin xyz="0 0 0" rpy="0 0 0" />
 			<geometry name="pioneer_geom">
 				<mesh filename="package://p3dx_description/meshes/center_hubcap.stl" />
 			</geometry>
-			<material name="swivel">
-				<color rgba="0.5 0.5 0.5 1" />
-			</material>
-		</visual>
-		<collision>
-			<origin xyz="0 0 0" rpy="0 0 0" />
-			<geometry>
-				<box size="0 0 0" />
-			</geometry>
-		</collision>
-	</link>
-	<joint name="swivel_hubcap_joint" type="continuous">
+			<material name="swivel"></material>
+		</visual>
+		<collision>
+			<origin xyz="0 0 0" rpy="0 0 0" />
+			<geometry>
+				<box size="0.00001 0.00001 0.00001" />
+			</geometry>
+		</collision>
+	</link>
+	<joint name="swivel_hubcap_joint" type="fixed">
 		<origin xyz="-0.026 0 -0.016" rpy="0 0 0" />
 		<axis xyz="0 1 0" />
@@ -148,23 +130,20 @@
 		<child link="center_wheel" />
 	</joint>
-  <!-- center_wheel -->
+	<!-- center_wheel -->
 	<link name="center_wheel">
 		<inertial>
-			<mass value="0.1" />
-			<origin xyz="0 0 0" />
-			<inertia ixx="0.012411765597" ixy="-0.000711733678" ixz="0.00050272983"
-				iyy="0.015218160428" iyz="-0.000004273467" izz="0.011763977943" />
-		</inertial>
-		<visual name="base_visual">
+			<mass value="1.0" />
+			<origin xyz="0 0 0" />
+			<inertia ixx="0.012411765597" ixy="-0.000711733678" ixz="0.00050272983" iyy="0.015218160428" iyz="-0.000004273467" izz="0.011763977943" />
+		</inertial>
+		<visual>
 			<origin xyz="0 0 0" rpy="0 0 0" />
 			<geometry name="pioneer_geom">
 				<mesh filename="package://p3dx_description/meshes/center_wheel.stl" />
 			</geometry>
-			<material name="WheelBlack">
-				<color rgba="0.117 0.117 0.117 1" />
-			</material>
-		</visual>
-		<collision>
-			<origin xyz="0 0 0" rpy="-1.57079635 0 0" />
+			<material name="WheelBlack"></material>
+		</visual>
+		<collision>
+			<origin xyz="0 0 0" rpy="${-3.1415927/2.0} 0 0" />
 			<geometry>
 				<cylinder radius="0.0375" length="0.01" />
@@ -177,56 +156,13 @@
 		<child link="center_hubcap"/>
 	</joint>
-	<xacro:p3dx_wheel suffix="left" parent="chassis" reflect="1"/>
-	<xacro:p3dx_wheel suffix="right" parent="chassis" reflect="-1"/>
-	<link name="rplidar">
-		<inertial>            <!--Inertial valuse include origin, mass and inertias as per CAD model-->
-		<mass value="0.10441" />
-		<origin rpy="0 0 0" xyz="0 0 0" />
-		<inertia ixx="0.1000000042" ixy="0" ixz="0" iyy="0.1000000042" iyz="0" izz="0.1000000040" /> <!-- Taken at the output coordinate system-->
-		</inertial>
-		<collision>           <!-- Collision values include dimensions and origin-->
-		<origin rpy="0 0 0" xyz="0 0 0" />
-		<geometry>
-			<mesh filename="package://p3dx_description/meshes/rplidar.dae" scale="1 1 1"/>
-		</geometry>
-		</collision>
-		<visual>               <!-- Visual valuse include origin, material and mesh to make model look similar to real robot-->
-		<origin rpy="0 0 0" xyz="0 0 0" />
-		<geometry>
-			<mesh filename="package://p3dx_description/meshes/rplidar.dae" scale="1 1 1"/>
-		</geometry>
-		<material name="RPLidarBlack">
-			<color rgba="0.117 0.117 0.117 1" />
-		</material>
-		</visual>
-  </link>
-   <joint name="chassis_to_rplidar" type="fixed">
-     <axis xyz="0 0 0" />
-     <origin rpy="0 0 -1.57" xyz="0.06 0.0 0.33" />
-     <parent link="chassis" />
-     <child link="rplidar" />
-   </joint>
-	<!--Lidar-->
-  	<!-- <xacro:m_link_cylinder name="rplidar"
-                   origin_rpy="0 0 0" origin_xyz="0 0 0"
-                   mass="0.10441"
-                   ixx="0.1000000042" ixy="0" ixz="0"
-                   iyy="0.1000000042" iyz="0"
-                   izz="0.1000000040"
-                   material="black"
-                   filename="package://wheelchair_description/meshes/rplidar.dae" scale="1 1 1"/> -->
-	<!-- joint between chassis and lidar -->
-    <!-- <xacro:f_joint name="chassis_to_rplidar"
-			type="fixed"
-			axis_xyz="0 0 0"
-			origin_rpy="0 0 -1.57" origin_xyz="0.23 0 -0.15"
-			parent="chassis" child="rplidar" /> -->
-	<xacro:sensor_d435 parent="chassis">
-		<origin xyz="0.1 0 0.860" rpy="0 0 0"/>
-    </xacro:sensor_d435>
-	<!-- <xacro:sensor_d455 parent="chassis" use_nominal_extrinsics="$(arg use_nominal_extrinsics)">
-		<origin xyz="0 0 0" rpy="0 0 0"/>
-	</xacro:sensor_d455> -->
-  <!-- front_sonar -->
+	<!-- End of Legacy for diff drive plugin
+	https://github.com/ros-simulation/gazebo_ros_pkgs/pull/707/files
+	"This setting assumes you have a old package, where the right and left wheel are changed to fix a former code issue\n"
+	"To get rid of this error just set <legacyMode> to false if you just created a new package.\n"
+	"To fix an old package you have to exchange left wheel by the right wheel.\n"
+	-->
+	<xacro:p3dx_wheel suffix="left" parent="base_link" reflect="-1"/>
+	<xacro:p3dx_wheel suffix="right" parent="base_link" reflect="1"/>
+	<!-- front_sonar -->
 	<link name="front_sonar">
 		<inertial>
@@ -235,17 +171,15 @@
 			<inertia ixx="1" ixy="0" ixz="0" iyy="1" iyz="0" izz="1" />
 		</inertial>
-		<visual name="front_sonar_vis">
+		<visual>
 			<origin rpy="0 0 0" xyz="0 0 0" />
 			<geometry name="pioneer_geom">
 				<mesh filename="package://p3dx_description/meshes/front_sonar.stl" />
 			</geometry>
-			<material name="SonarYellow">
-				<color rgba="0.715 0.583 0.210 1.0" />
-			</material>
+			<material name="SonarYellow"></material>
 		</visual>
 		<collision>
 			<origin rpy="0 0 0" xyz="0 0 0" />
 			<geometry>
-				<box size="0 0 0" />
+				<box size="0.00001 0.00001 0.00001" />
 			</geometry>
 		</collision>
@@ -253,5 +187,5 @@
 	<joint name="base_front_joint" type="fixed">
 		<origin rpy="0 0 0" xyz="0.109 0 0.209" />
-		<parent link="chassis" />
+		<parent link="base_link" />
 		<child link="front_sonar" />
 	</joint>
@@ -278,6 +212,6 @@
 	<joint name="lms100_joint" type="fixed">
 		<axis xyz="0 1 0" />
-		<origin xyz="0.16 0 0.15" rpy="0 0 0" />
-		<parent link="chassis" />
+		<origin xyz="0.12 0 0.26" rpy="0 0 0" />
+		<parent link="base_link" />
 		<child link="lms100" />
 	</joint>

File: src/p3dx_description/urdf/pioneer3dx_wheel.xacro (robot description, xacro)
@@ -18,5 +18,5 @@
 <robot xmlns:xacro="http://ros.org/wiki/xacro">
 	<!-- properties (constants) -->
-	<property name="M_PI" value="3.14159" />
+	<xacro:property name="M_PI" value="3.14159" />
 	<!-- right/left hubcap + wheel -->
 	<xacro:macro name="p3dx_wheel" params="suffix parent reflect">
@@ -26,15 +26,12 @@
 				<mass value="0.5" />
 				<origin xyz="0 0 0" />
-				<inertia ixx="0.012411765597" ixy="0" ixz="0" iyy="0.015218160428"
-					iyz="0" izz="0.011763977943" />
+				<inertia ixx="0.012411765597" ixy="0" ixz="0" iyy="0.015218160428" iyz="0" izz="0.011763977943" />
 			</inertial>
-			<visual name="base_visual">
+			<visual>
 				<origin xyz="0 0 0" rpy="0 0 0" />
 				<geometry name="pioneer_geom">
 					<mesh filename="package://p3dx_description/meshes/${suffix}_wheel.stl" />
 				</geometry>
-				<material name="WheelBlack">
-					<color rgba="0.117 0.117 0.117 1" />
-				</material>
+				<material name="WheelBlack"></material>
 			</visual>
 			<collision>
@@ -56,20 +53,17 @@
 				<mass value="0.01" />
 				<origin xyz="0 0 0" />
-				<inertia ixx="0.012411765597" ixy="0" ixz="0" iyy="0.015218160428"
-					iyz="0" izz="0.011763977943" />
+				<inertia ixx="0.012411765597" ixy="0" ixz="0" iyy="0.015218160428" iyz="0" izz="0.011763977943" />
 			</inertial>
-			<visual name="base_visual">
+			<visual>
 				<origin xyz="0 0 0" rpy="0 0 0" />
 				<geometry name="pioneer_geom">
 					<mesh filename="package://p3dx_description/meshes/${suffix}_hubcap.stl" />
 				</geometry>
-				<material name="HubcapYellow">
-					<color rgba="1.0 0.811 0.151 1.0" />
-				</material>
+				<material name="HubcapYellow"></material>
 			</visual>
 			<collision>
 				<origin xyz="0 0 0" rpy="0 0 0" />
 				<geometry>
-					<box size="0 0 0" />
+					<box size="0.00001 0.00001 0.00001" />
 				</geometry>
 			</collision>
@@ -81,16 +75,18 @@
 			<joint_properties damping="0.0" friction="0.0" />
 			<origin xyz="0 ${reflect*0.158} 0.091" rpy="0 0 0" />
-			<parent link="chassis" />
+			<parent link="base_link" />
 			<child link="p3dx_${suffix}_wheel" />
 		</joint>
 		<!-- gazebo elements -->
-    <transmission name="${parent}_${suffix}_wheel_trans">
-      <type>pr2_mechanism_model/SimpleTransmission</type>
-      <joint name="base_${suffix}_wheel_joint" />
-      <actuator name="base_${suffix}_wheel_motor">
-        <hardwareInterface>EffortJointInterface</hardwareInterface>
-        <mechanicalReduction>${reflect * 624/35 * 80/19}</mechanicalReduction>
-      </actuator>
-    </transmission>
+		<transmission name="${parent}_${suffix}_wheel_trans">
+			<type>pr2_mechanism_model/SimpleTransmission</type>
+			<joint name="base_${suffix}_wheel_joint">
+				<hardwareInterface>hardware_interface/EffortJointInterface</hardwareInterface>
+			</joint>
+			<actuator name="base_${suffix}_wheel_motor">
+				<hardwareInterface>EffortJointInterface</hardwareInterface>
+				<mechanicalReduction>${reflect * 624/35 * 80/19}</mechanicalReduction>
+			</actuator>
+		</transmission>
 		<gazebo reference="p3dx_${suffix}_hubcap">
 			<material>Gazebo/Yellow</material>
